File: Issue_6/Issue_6.kicad_sch (KiCad schematic)
At the start: 289 parts, among them IC1 4164A, IC10 4164A, IC11 4164A, IC12 4164A, IC13 4164A, IC14 4164A, IC15 4164A, IC16 4164A, IC18 68008D, IC19 74LS257, IC2 4164A, IC20 74LS257, IC21 74LS245, IC22 ZX8301, IC23 ZX8302, IC24 8749, IC25 MC1488, IC26 MC1489, IC28 MC1377P, IC29 2G007, IC3 4164A, IC30 2G007, IC31 LM7805_TO220, IC32 LM7805_TO220, IC33 27256, IC34 27128, IC36 L7912, IC37 L7812, IC38 GAL16V8, IC4 4164A, IC5 4164A, IC6 4164A, IC7 4164A, IC8 4164A, IC9 4164A, J1 QL_SLOT_DIN41612, J10 AudioJack2_Ground_Switch, J101 Conn_01x07, J102 Conn_01x07, J11 Conn_01x09_Socket, J12 Conn_01x11_Socket, J2 QL_cartridge_ROM, J201 Conn_01x07, J202 Conn_01x07, J3 Conn_01x06, J4 Conn_01x06, J5 Conn_01x06, J6 Conn_01x06, J7 DIN-8, J8 Conn_01x03_Pin, J9 AudioJack2_Ground_Switch, M1 UM1233, M2 Motor_DC, M3 Motor_DC, SW1 SW_SPDT, SW2 SW_SPDT, U35 LM7805_TO220, X1 15Mhz, X2 32768Khz, X3 4.4336Mhz, X4 11Mhz

Commit message: aestetical
Parts:
- D20_1, D21_1, D27_2, R47, R92_2: now not fitted
Changed lines of the file:
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@@
 		(in_bom yes)
 		(on_board yes)
-		(dnp no)
+		(dnp yes)
 		(property "Reference" "R92_2"
 			(at 154.94 506.7299 0)
@@
 		(in_bom yes)
 		(on_board yes)
-		(dnp no)
+		(dnp yes)
 		(fields_autoplaced yes)
 		(property "Reference" "D27_2"
@@
 		(in_bom yes)
 		(on_board yes)
-		(dnp no)
+		(dnp yes)
 		(fields_autoplaced yes)
 		(property "Reference" "R47"
@@
 		(in_bom yes)
 		(on_board yes)
-		(dnp no)
+		(dnp yes)
 		(property "Reference" "D21_1"
 			(at 624.586 215.646 0)
@@
 		(in_bom yes)
 		(on_board yes)
-		(dnp no)
+		(dnp yes)
 		(property "Reference" "D20_1"
 			(at 445.262 216.408 0)
