File: Issue_7ALEA/Issue_7ALEA.kicad_sch (KiCad schematic)
At the start: 289 parts, among them IC1 4164A, IC10 4164A, IC11 4164A, IC12 4164A, IC13 4164A, IC14 4164A, IC15 4164A, IC16 4164A, IC18 68008D, IC19 74LS257, IC2 4164A, IC20 74LS257, IC21 74LS245, IC22 ZX8301, IC23 ZX8302, IC24 8749, IC25 MC1488, IC26 MC1489, IC28 MC1377P, IC29 2G007, IC3 4164A, IC30 2G007, IC31 LM7805_TO220, IC32 LM7805_TO220, IC33 27256, IC34 27128, IC36 L7912, IC37 L7812, IC38 GAL16V8, IC4 4164A, IC5 4164A, IC6 4164A, IC7 4164A, IC8 4164A, IC9 4164A, J1 QL_SLOT_DIN41612, J10 AudioJack2_Ground_Switch, J101 Conn_01x07, J102 Conn_01x07, J11 Conn_01x09_Socket, J12 Conn_01x11_Socket, J2 QL_cartridge_ROM, J201 Conn_01x07, J202 Conn_01x07, J3 Conn_01x06, J4 Conn_01x06, J5 Conn_01x06, J6 Conn_01x06, J7 DIN-8, J8 Conn_01x03_Pin, J9 AudioJack2_Ground_Switch, M1 UM1233, M2 Motor_DC, M3 Motor_DC, SW1 SW_SPDT, SW2 SW_SPDT, U35 LM7805_TO220, X1 15Mhz, X2 32768Khz, X3 4.4336Mhz, X4 11Mhz

Commit message: small updates to issue 5
Parts:
- removed R102, R103: 0, 8bits:R_Axial_DIN0207_L6.3mm_D2.5mm_P12.7mm_Horizontal_W, symbol Device:R
- added D18, D19, D24, D30, D31: 5V1, Diode_THT:D_DO-34_SOD68_P2.54mm_Vertical_KathodeUp, symbol Device:D_Zener_Small
Connections:
- net BLUE: now also D18.1 (K)
- net CSYNC: now also D30.1 (K)
- net GND: now also D18.2 (A), D19.2 (A), D24.2 (A), D30.2 (A), D31.2 (A)
- net GREEN: now also D19.1 (K)
- net RAW1: now also IC23.21 (RAW1)
- net RAW2: now also IC23.19 (RAW2)
- net RED: now also D24.1 (K)
- net VSYNC: now also D31.1 (K)
Other:
- note removed: "NOTE: R107,R108 Aereal instalation over IC23 an a wire to -12V (PIN 1 of IC25)"
- moved on the sheet: R107, R108
